File: pcb/hackpad copy.kicad_pcb (KiCad board)
At the start: 2 copper layers, 94.3 x 68.9 mm, 28 parts, among them J2 OLED_128x32, SW1 SW_Push_45deg, SW2 SW_Push_45deg, SW3 SW_Push_45deg, SW4 SW_Push_45deg, SW5 SW_Push_45deg, SW6 SW_Push_45deg, SW7 SW_Push_45deg, SW8 SW_Push_45deg, SW9 RotaryEncoder_Switch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

Commit message: Add files via upload
Parts:
- removed D12: Diode, Diode_THT:D_DO-35_SOD27_P7.62mm_Horizontal
Connections:
- SW1 pad 1: RINPUT -> col1
- SW4 pad 1: RINPUT -> col1
- SW9 pad S1: RINPUT -> unconnected-(SW9-PadS1)
- SW9 pad S2: ROUTPUT -> unconnected-(SW9-PadS2)
- U1 pad 4: RINPUT -> col1
Routing:
- net RINPUT: track 125.0 -> 0.00 mm, vias 1 -> 0
- net row1: track 121.8 -> 70.9 mm, vias 4 -> 3
- net col1: track 0.00 -> 44.7 mm, vias 0 -> 1
- net ROUTPUT: track 20.6 -> 0.00 mm
- added copper zone on B.Cu, net (none)
- added copper zone on F.Cu, net (none)
Other:
- board text added: "blipblip"
