File: pcb/hackpad copy.kicad_sch (KiCad schematic)
At the start: 28 parts, among them J2 OLED_128x32, SW1 SW_Push_45deg, SW2 SW_Push_45deg, SW3 SW_Push_45deg, SW4 SW_Push_45deg, SW5 SW_Push_45deg, SW6 SW_Push_45deg, SW7 SW_Push_45deg, SW8 SW_Push_45deg, SW9 RotaryEncoder_Switch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

Commit message: Add files via upload
Parts:
- removed D12: Diode, Diode_THT:D_DO-35_SOD27_P7.62mm_Horizontal, symbol ScottoKeebs:Placeholder_Diode
Connections:
- net RINPUT renamed col1
- net col1: no longer SW9.S1
- net ROUTPUT: no longer names the net of SW9.S2
